File: pcb/credit_board.sch (KiCad schematic (older format))
At the start: 11 parts, among them J1 Conn_01x05_Male, J2 Conn_01x03_Male, J3 Jack-DC, U1 74HC04, Y1 10MHz, Y2 32.768 kHz

Commit message: no connected pins are pull up by 10k resistors.
Parts:
- added J4, J5, J6: pull-up, PINHEADER:PINHEADER_1x1, symbol Conn_01x01_Male
- added R4, R5, R6: 10k, Resistors_THT:R_Axial_DIN0204_L3.6mm_D1.6mm_P2.54mm_Vertical, symbol R
- U1: footprint (none) -> Housings_DIP:DIP-14_W7.62mm
Connections:
- wire segments 55 -> 60
Other:
- moved on the sheet: C1, C2, J2, R1, U1D, U1E, U1F, Y1

Commit message: 74HC04 の input に未接続の端子は，pull up するようにした。
Parts:
- removed J4: pull-up, PINHEADER:PINHEADER_1x1, symbol Conn_01x01_Male
- added J?: pull-up, PINHEADER:PINHEADER_1x1, symbol Conn_01x01_Male
- added JP? (x3): amp, symbol Jumper_NO_Small
- added JP? (x3): pull up, symbol Jumper_NO_Small
- J1: value Conn_01x05_Male -> amp&pull-up
Connections:
- net labels added: out
- wire segments 60 -> 80
Other:
- moved on the sheet: J2, J5, J6, R2, R3, R4, R5, R6, U1A, U1B, U1C, U1D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

Commit message: completed to make a initial credit board.
Parts:
- removed J1: amp&pull-up, PINHEADER:PINHEADER_1x5, symbol Conn_01x05_Male
- removed J?: pull-up, PINHEADER:PINHEADER_1x1, symbol Conn_01x01_Male
- removed JP? (x3): amp, symbol Jumper_NO_Small
- removed JP? (x3): pull up, symbol Jumper_NO_Small
- added J1, J4: amp or pull-up, PINHEADER:PINHEADER_1x3, symbol Conn_01x03_Male
- J2: value Conn_01x03_Male -> amp or pull-up
- J5, J6: value pull-up -> clk
- Y2: footprint Crystals:Crystal_DS26_d2.0mm_l6.0mm_Horizontal -> Crystals:Crystal_AT310_d3.0mm_l10.0mm_Vertical
Connections:
- net labels removed: out
- wire segments 80 -> 54
Other:
- note added: "clock"
- moved on the sheet: J2, R4, R5, R6, U1C, U1D

Commit message: 本当の，本当に完成したよぉぉぉぉ。
神経質には完成させられないんじゃないだろうか？と完成を危ぶんだこともありました。
しかし，なんとか完成しました。
めでたし。めでたし。
Parts:
- J1, J2, J4: footprint PINHEADER:PINHEADER_1x3 -> Pin_Headers:Pin_Header_Straight_1x03_Pitch2.54mm
- J5, J6: footprint PINHEADER:PINHEADER_1x1 -> Connectors:Pin_d1.0mm_L10.0mm
- R4, R5, R6: footprint Resistors_THT:R_Axial_DIN0204_L3.6mm_D1.6mm_P2.54mm_Vertical -> Resistors_THT:R_Axial_DIN0207_L6.3mm_D2.5mm_P2.54mm_Vertical
- U1: symbol 74HC04 -> 74HC04-RESCUE-credit_board
Changed lines of the file:
@@
 EESchema Schematic File Version 2
+LIBS:credit_board-rescue
 LIBS:74xgxx
 LIBS:74xx
 LIBS:Altera
 LIBS:ESD_Protection
-LIBS:LEM
 LIBS:Lattice
 LIBS:Oscillators
 LIBS:Power_Management
-LIBS:RFSolutions
 LIBS:Worldsemi
 LIBS:Xicor
@@
 LIBS:battery_management
 LIBS:bbd
-LIBS:bosch
 LIBS:brooktre
 LIBS:cmos4000
@@
 LIBS:diode
 LIBS:display
-LIBS:driver_gate
 LIBS:dsp
 LIBS:elec-unifil
 LIBS:ftdi
 LIBS:gennum
-LIBS:graphic_symbols
 LIBS:hc11
-LIBS:infineon
 LIBS:intel
 LIBS:interface
-LIBS:intersil
 LIBS:ir
-LIBS:leds
 LIBS:linear
-LIBS:logic_programmable
 LIBS:maxim
 LIBS:mechanical
@@
 LIBS:microchip_pic16mcu
 LIBS:microchip_pic18mcu
-LIBS:microchip_pic24mcu
 LIBS:microchip_pic32mcu
 LIBS:microcontrollers
-LIBS:modules
 LIBS:motor_drivers
 LIBS:motorola
@@
 LIBS:msp430
 LIBS:nordicsemi
-LIBS:nxp
 LIBS:nxp_armmcu
 LIBS:onsemi
@@
 LIBS:transf
 LIBS:transistors
-LIBS:triac_thyristor
 LIBS:ttl_ieee
 LIBS:valves
@@
 $EndComp
 $Comp
-L 74HC04 U1
+L 74HC04-RESCUE-credit_board U1
 U 1 1 59C5818C
 P 4950 4350
@@
 $EndComp
 $Comp
-L 74HC04 U1
+L 74HC04-RESCUE-credit_board U1
 U 5 1 59C581BD
 P 5950 1700
@@
 $EndComp
 $Comp
-L 74HC04 U1
+L 74HC04-RESCUE-credit_board U1
 U 6 1 59C58206
 P 4900 1700
@@
 $EndComp
 $Comp
-L 74HC04 U1
+L 74HC04-RESCUE-credit_board U1
 U 2 1 59C58651
 P 6550 4350
@@
 $EndComp
 $Comp
-L 74HC04 U1
+L 74HC04-RESCUE-credit_board U1
 U 3 1 59C5869C
 P 7550 4350
@@
 $EndComp
 $Comp
-L 74HC04 U1
+L 74HC04-RESCUE-credit_board U1
 U 4 1 59C586F5
 P 6950 1700
@@
 F 0 "J2" H 6450 2250 50  0000 C CNN
 F 1 "amp or pull-up" V 6350 2050 50  0000 C CNN
-F 2 "PINHEADER:PINHEADER_1x3" H 6450 2050 50  0001 C CNN
+F 2 "Pin_Headers:Pin_Header_Straight_1x03_Pitch2.54mm" H 6450 2050 50  0001 C CNN
 F 3 "" H 6450 2050 50  0001 C CNN
 	1    6450 2050
@@
 $EndComp
 $Comp
-L 74HC04 U1
+L 74HC04-RESCUE-credit_board U1
 U 7 1 59C5C494
 P 3600 3050
@@
 F 0 "R5" V 6550 1450 50  0000 C CNN
 F 1 "10k" V 6450 1450 50  0000 C CNN
-F 2 "Resistors_THT:R_Axial_DIN0204_L3.6mm_D1.6mm_P2.54mm_Vertical" V 6480 1450 50  0001 C CNN
+F 2 "Resistors_THT:R_Axial_DIN0207_L6.3mm_D2.5mm_P2.54mm_Vertical" V 6480 1450 50  0001 C CNN
 F 3 "" H 6550 1450 50  0001 C CNN
 	1    6550 1450
@@
 F 0 "R4" V 6150 4050 50  0000 C CNN
 F 1 "10k" V 6250 4050 50  0000 C CNN
-F 2 "Resistors_THT:R_Axial_DIN0204_L3.6mm_D1.6mm_P2.54mm_Vertical" V 6080 4050 50  0001 C CNN
+F 2 "Resistors_THT:R_Axial_DIN0207_L6.3mm_D2.5mm_P2.54mm_Vertical" V 6080 4050 50  0001 C CNN
 F 3 "" H 6150 4050 50  0001 C CNN
 	1    6150 4050
@@
 F 0 "R6" V 7150 4050 50  0000 C CNN
 F 1 "10k" V 7050 4050 50  0000 C CNN
-F 2 "Resistors_THT:R_Axial_DIN0204_L3.6mm_D1.6mm_P2.54mm_Vertical" V 7080 4050 50  0001 C CNN
+F 2 "Resistors_THT:R_Axial_DIN0207_L6.3mm_D2.5mm_P2.54mm_Vertical" V 7080 4050 50  0001 C CNN
 F 3 "" H 7150 4050 50  0001 C CNN
 	1    7150 4050
@@
 F 0 "J1" H 6150 5700 50  0000 C CNN
 F 1 "amp or pull-up" V 6000 5500 50  0000 C CNN
-F 2 "PINHEADER:PINHEADER_1x3" H 6050 5500 50  0001 C CNN
+F 2 "Pin_Headers:Pin_Header_Straight_1x03_Pitch2.54mm" H 6050 5500 50  0001 C CNN
 F 3 "" H 6050 5500 50  0001 C CNN
 	1    6050 5500
@@
 F 0 "J4" H 7150 5700 50  0000 C CNN
 F 1 "amp or pull-up" V 7000 5500 50  0000 C CNN
-F 2 "PINHEADER:PINHEADER_1x3" H 7050 5500 50  0001 C CNN
+F 2 "Pin_Headers:Pin_Header_Straight_1x03_Pitch2.54mm" H 7050 5500 50  0001 C CNN
 F 3 "" H 7050 5500 50  0001 C CNN
 	1    7050 5500
@@
 F 0 "J6" H 7950 4100 50  0000 C CNN
 F 1 "clk" H 7900 4000 50  0000 C CNN
-F 2 "PINHEADER:PINHEADER_1x1" H 7950 4050 50  0001 C CNN
+F 2 "Connectors:Pin_d1.0mm_L10.0mm" H 7950 4050 50  0001 C CNN
 F 3 "" H 7950 4050 50  0001 C CNN
 	1    7950 4050
@@
 F 0 "J5" H 7350 1450 50  0000 C CNN
 F 1 "clk" H 7300 1350 50  0000 C CNN
-F 2 "PINHEADER:PINHEADER_1x1" H 7350 1400 50  0001 C CNN
+F 2 "Connectors:Pin_d1.0mm_L10.0mm" H 7350 1400 50  0001 C CNN
 F 3 "" H 7350 1400 50  0001 C CNN
 	1    7350 1400

Commit message: board の clock 部は完成。
Parts:
- renumbered J3 to J1, J1 to J2, J2 to J3, R2 to R1, R1 to R2
Connections:
- net at R1.2, Y2.1: now also U1.13; no longer U1.1
- net output1: now reaches J2.1 (Pin_1), R3.2, Y2.2
- net at R1.1, R3.1: now also U1.12; no longer U1.2
- net at C1.1, R2.2, Y1.1: now also U1.1; no longer U1.13
- net at C2.1, R2.1, Y1.2: now also U1.2, U1.3; no longer U1.11, U1.12
- net amp2: now reaches U1.10
- net amp2: now also J4.1 (Pin_1); no longer J3.1 (Pin_1)
- net amp1: now reaches J2.2 (Pin_2)
- net amp1: now also U1.11; no longer U1.3
- net amp3: now reaches U1.4
- net amp3: now also J3.1 (Pin_1); no longer J4.1 (Pin_1)
- net at U1.5: now also J3.2 (Pin_2); no longer J4.2 (Pin_2)
- net output2: now reaches J6.1 (Pin_1)
- net output2: now also U1.8; no longer U1.6
- net output3: now reaches J5.1 (Pin_1)
- net output3: now also U1.6; no longer U1.8
- net at U1.9: now also J4.2 (Pin_2); no longer J3.2 (Pin_2)
- net pull-up3: now reaches J3.3 (Pin_3), R5.1
- net pull-up1: now reaches J2.3 (Pin_3), R4.1
- net pull-up2: now reaches J4.3 (Pin_3), R6.1
Other:
- moved on the sheet: C1, C2, J2, J3, J4, J5, J6, R1, R2, R3, R4, R5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

Commit message: Jack-DCの3PINを未接続にした。
Parts:
- removed Y1: 10MHz, Crystals:Crystal_HC50_Vertical, symbol Crystal
- removed Y2: 32.768 kHz, Crystals:Crystal_AT310_d3.0mm_l10.0mm_Vertical, symbol Crystal
- added J7: 32.768kHz xtal, PINHEADER:PINHEADER_1x2, symbol Conn_01x02_Female
- added J8: 10MHz xtal, PINHEADER:PINHEADER_1x3, symbol Conn_01x03_Female
- R1, R2, R3, R4, R5, R6: footprint Resistors_THT:R_Axial_DIN0207_L6.3mm_D2.5mm_P2.54mm_Vertical -> Resistors_THT:R_Axial_DIN0207_L6.3mm_D2.5mm_P7.62mm_Horizontal
- U1: footprint Housings_DIP:DIP-14_W7.62mm -> IC:SN74HC04N
Connections:
- wire segments 54 -> 53
- no-connect marks 0 -> 2
Changed lines of the file:
@@
 LIBS:Altera
 LIBS:ESD_Protection
-LIBS:LEM
 LIBS:Lattice
 LIBS:Oscillators
 LIBS:Power_Management
-LIBS:RFSolutions
 LIBS:Worldsemi
 LIBS:Xicor
@@
 LIBS:diode
 LIBS:display
-LIBS:driver_gate
 LIBS:dsp
 LIBS:elec-unifil
 LIBS:ftdi
 LIBS:gennum
-LIBS:graphic_symbols
 LIBS:hc11
-LIBS:infineon
 LIBS:intel
 LIBS:interface
-LIBS:intersil
 LIBS:ir
 LIBS:leds
 LIBS:linear
-LIBS:logic_programmable
 LIBS:maxim
 LIBS:mechanical
@@
 $EndDescr
 $Comp
-L Crystal Y2
-U 1 1 59C473F7
-P 5100 3050
-F 0 "Y2" H 5100 3200 50  0000 C CNN
-F 1 "32.768 kHz" H 5100 2900 50  0000 C CNN
-F 2 "Crystals:Crystal_AT310_d3.0mm_l10.0mm_Vertical" H 5100 3050 50  0001 C CNN
-F 3 "" H 5100 3050 50  0000 C CNN
-	1    5100 3050
-	1    0    0    -1
-$EndComp
-$Comp
 L R R1
 U 1 1 59C47429
@@
 F 0 "R1" V 5050 2550 50  0000 C CNN
 F 1 "10MΩ" V 4950 2550 50  0000 C CNN
-F 2 "Resistors_THT:R_Axial_DIN0207_L6.3mm_D2.5mm_P2.54mm_Vertical" V 4980 2550 50  0001 C CNN
+F 2 "Resistors_THT:R_Axial_DIN0207_L6.3mm_D2.5mm_P7.62mm_Horizontal" V 4980 2550 50  0001 C CNN
 F 3 "" H 5050 2550 50  0000 C CNN
 	1    5050 2550
@@
 $EndComp
 $Comp
-L Crystal Y1
-U 1 1 59C47EFB
-P 5050 4650
-F 0 "Y1" H 5050 4800 50  0000 C CNN
-F 1 "10MHz" H 5050 4500 50  0000 C CNN
-F 2 "Crystals:Crystal_HC50_Vertical" H 5050 4650 50  0001 C CNN
-F 3 "" H 5050 4650 50  0000 C CNN
-	1    5050 4650
-	1    0    0    -1
-$EndComp
-$Comp
 L R R2
 U 1 1 59C47F01
@@
 F 0 "R2" V 5130 3950 50  0000 C CNN
 F 1 "1MΩ" V 5050 3950 50  0000 C CNN
-F 2 "Resistors_THT:R_Axial_DIN0207_L6.3mm_D2.5mm_P2.54mm_Vertical" V 4980 3950 50  0001 C CNN
+F 2 "Resistors_THT:R_Axial_DIN0207_L6.3mm_D2.5mm_P7.62mm_Horizontal" V 4980 3950 50  0001 C CNN
 F 3 "" H 5050 3950 50  0000 C CNN
 	1    5050 3950
@@
 F 0 "R3" V 5600 2750 50  0000 C CNN
 F 1 "470kΩ" V 5500 2750 50  0000 C CNN
-F 2 "Resistors_THT:R_Axial_DIN0207_L6.3mm_D2.5mm_P2.54mm_Vertical" V 5530 2750 50  0001 C CNN
+F 2 "Resistors_THT:R_Axial_DIN0207_L6.3mm_D2.5mm_P7.62mm_Horizontal" V 5530 2750 50  0001 C CNN
 F 3 "" H 5600 2750 50  0000 C CNN
 	1    5600 2750
@@
 F 0 "U1" H 5200 4400 50  0000 C CNN
 F 1 "74HC04" H 5250 4200 50  0000 C CNN
-F 2 "Housings_DIP:DIP-14_W7.62mm" H 5050 4300 50  0001 C CNN
+F 2 "IC:SN74HC04N" H 5050 4300 50  0001 C CNN
 F 3 "" H 5050 4300 50  0000 C CNN
 	1    5050 4300
@@
 F 0 "U1" H 6850 2300 50  0000 C CNN
 F 1 "74HC04" H 6900 2400 50  0000 C CNN
-F 2 "Housings_DIP:DIP-14_W7.62mm" H 6700 2200 50  0001 C CNN
+F 2 "IC:SN74HC04N" H 6700 2200 50  0001 C CNN
 F 3 "" H 6700 2200 50  0000 C CNN
 	5    6700 2200
@@
 F 0 "U1" H 5250 2300 50  0000 C CNN
 F 1 "74HC04" H 5300 2100 50  0000 C CNN
-F 2 "Housings_DIP:DIP-14_W7.62mm" H 5100 2200 50  0001 C CNN
+F 2 "IC:SN74HC04N" H 5100 2200 50  0001 C CNN
 F 3 "" H 5100 2200 50  0000 C CNN
 	6    5100 2200
@@
 F 0 "U1" H 6250 4400 50  0000 C CNN
 F 1 "74HC04" H 6300 4200 50  0000 C CNN
-F 2 "Housings_DIP:DIP-14_W7.62mm" H 6100 4300 50  0001 C CNN
+F 2 "IC:SN74HC04N" H 6100 4300 50  0001 C CNN
 F 3 "" H 6100 4300 50  0000 C CNN
 	2    6100 4300
@@
 F 0 "U1" H 7250 4400 50  0000 C CNN
 F 1 "74HC04" H 7300 4200 50  0000 C CNN
-F 2 "Housings_DIP:DIP-14_W7.62mm" H 7100 4300 50  0001 C CNN
+F 2 "IC:SN74HC04N" H 7100 4300 50  0001 C CNN
 F 3 "" H 7100 4300 50  0000 C CNN
 	3    7100 4300
@@
 F 0 "U1" H 7850 2300 50  0000 C CNN
 F 1 "74HC04" H 7900 2100 50  0000 C CNN
-F 2 "Housings_DIP:DIP-14_W7.62mm" H 7700 2200 50  0001 C CNN
+F 2 "IC:SN74HC04N" H 7700 2200 50  0001 C CNN
 F 3 "" H 7700 2200 50  0000 C CNN
 	4    7700 2200
@@
 F 0 "U1" H 3600 3100 50  0000 C CNN
 F 1 "74HC04" H 3600 3000 50  0000 C CNN
-F 2 "Housings_DIP:DIP-14_W7.62mm" H 3600 3050 50  0001 C CNN
+F 2 "IC:SN74HC04N" H 3600 3050 50  0001 C CNN
 F 3 "" H 3600 3050 50  0001 C CNN
 	7    3600 3050
@@
 F 0 "R5" V 6700 4050 50  0000 C CNN
 F 1 "10k" V 6600 4050 50  0000 C CNN
-F 2 "Resistors_THT:R_Axial_DIN0207_L6.3mm_D2.5mm_P2.54mm_Vertical" V 6630 4050 50  0001 C CNN
+F 2 "Resistors_THT:R_Axial_DIN0207_L6.3mm_D2.5mm_P7.62mm_Horizontal" V 6630 4050 50  0001 C CNN
 F 3 "" H 6700 4050 50  0001 C CNN
 	1    6700 4050
@@
 F 0 "R4" V 6300 1900 50  0000 C CNN
 F 1 "10k" V 6400 1900 50  0000 C CNN
-F 2 "Resistors_THT:R_Axial_DIN0207_L6.3mm_D2.5mm_P2.54mm_Vertical" V 6230 1900 50  0001 C CNN
+F 2 "Resistors_THT:R_Axial_DIN0207_L6.3mm_D2.5mm_P7.62mm_Horizontal" V 6230 1900 50  0001 C CNN
 F 3 "" H 6300 1900 50  0001 C CNN
 	1    6300 1900
@@
 F 0 "R6" V 7300 1900 50  0000 C CNN
 F 1 "10k" V 7200 1900 50  0000 C CNN
-F 2 "Resistors_THT:R_Axial_DIN0207_L6.3mm_D2.5mm_P2.54mm_Vertical" V 7230 1900 50  0001 C CNN
+F 2 "Resistors_THT:R_Axial_DIN0207_L6.3mm_D2.5mm_P7.62mm_Horizontal" V 7230 1900 50  0001 C CNN
 F 3 "" H 7300 1900 50  0001 C CNN
 	1    7300 1900
@@
 	8350 1150 6050 1150
 Wire Wire Line
-	4600 4650 4900 4650
+	4600 4650 4950 4650
 Wire Wire Line
 	4600 3950 4600 4650
@@
 	5600 2900 5600 3050
 Wire Wire Line
-	4600 3050 4950 3050
+	4600 3050 5050 3050
 Wire Wire Line
 	5200 2550 5600 2550
@@
 Wire Wire Line
 	4900 2550 4600 2550
-Wire Wire Line
-	2800 2750 2800 3050
 Connection ~ 2800 3250
 Connection ~ 2800 2800
@@
 	2800 3150 2800 3350
 Wire Wire Line
-	2800 3050 2900 3050
-Wire Wire Line
 	2900 3150 2800 3150
 Wire Wire Line
@@
 Wire Wire Line
 	2950 3550 2950 3250
-Connection ~ 2800 2950
 Wire Wire Line
 	5500 3950 5500 4650
@@
 	5250 5000 5250 4650
 Wire Wire Line
-	5500 4650 5200 4650
+	5500 4650 5150 4650
 Connection ~ 5250 4650
 Wire Wire Line
@@
 	7200 2200 7200 3150
 Wire Wire Line
-	5250 3050 6100 3050
+	5150 3050 6100 3050
 Wire Wire Line
 	6200 2200 6200 3150
@@
 Text Label 5900 3050 0    60   ~ 0
 output1
+$Comp
+L Conn_01x02_Female J7
+U 1 1 5A0855D5
+P 5050 2850
+F 0 "J7" H 5050 2950 50  0000 C CNN
+F 1 "32.768kHz xtal" V 4750 2850 50  0000 C CNN
+F 2 "PINHEADER:PINHEADER_1x2" H 5050 2850 50  0001 C CNN
+F 3 "" H 5050 2850 50  0001 C CNN
+	1    5050 2850
+	0    -1   -1   0
+$EndComp
+$Comp
+L Conn_01x03_Female J8
+U 1 1 5A085BCF
+P 5050 4850
+F 0 "J8" H 5050 5050 50  0000 C CNN
+F 1 "10MHz xtal" V 4750 4850 50  0000 C CNN
+F 2 "PINHEADER:PINHEADER_1x3" H 5050 4850 50  0001 C CNN
+F 3 "" H 5050 4850 50  0001 C CNN
+	1    5050 4850
+	0    1    1    0
+$EndComp
+NoConn ~ 5050 4650
+Wire Wire Line
+	2800 2750 2800 2950
+NoConn ~ 2900 3050
 $EndSCHEMATC
